File: motherboard.sch (EAGLE design)
At the start: 21 parts, among them IC1 LM2576, IC2 74LS595D, IC3 74LS595D, IC4 74LS595D, Q2 BSS84, U1 ATMEGA8U2AU, X1 USB_3PSHIELD-85-32003-00X-1, Y1 RES

Commit message: updated mobo sch
Parts:
- added C4: 100uF, adafruit:CPOL-US153CLV-0807
- added C5, C6, C7, C8, C9: 1uF, adafruit:C-USC1206
- added D2, D3: BAV199, diode:BAV199
- added IC5: VN5772AK, rov_club:VN5772AK
- added JP2: (no value), sparkfun:M02LOCK_LONGPADS
- added R6: 10k, adafruit:R-US_R1206
Connections:
- net SCL renamed !CLR
- removed net N$3: C1.+, IC1.IN, Q2.S, ZD1.C
- new net +12V: C1.+, C4.+, C5.1, D2.C, D3.C, IC1.IN, IC5.VCC@0, IC5.VCC@1, IC5.VCC@2, IC5.VCC@3, Q2.S, ZD1.C
- new net H1: IC5.IN1
- new net H2: IC5.IN2
- new net H3: IC5.IN3
- new net H4: IC5.IN4
- new net N$11: C6.1, D3.AC, IC5.DRAIN3@0, IC5.DRAIN3@1, IC5.DRAIN3@2, IC5.DRAIN3@3, IC5.SOURCE1@0, IC5.SOURCE1@1, JP2.1
- new net N$13: C6.2, D2.AC, IC5.DRAIN4@0, IC5.DRAIN4@1, IC5.DRAIN4@2, IC5.DRAIN4@3, IC5.SOURCE2@0, IC5.SOURCE2@1, JP2.2
- new net SENSE: IC5.SENSE, R6.1
- new net STAT: IC5.STAT3
- net +5V: now also C7.1, C8.1, C9.1
- net GND: now also C4.-, C5.2, C7.2, C8.2, C9.2, D2.A, D3.A, IC2.G, IC3.G, IC4.G, IC5.GND, IC5.SOURCE3@0, IC5.SOURCE3@1, IC5.SOURCE4@0, IC5.SOURCE4@1, R6.2
Other:
- moved on the sheet: IC3, IC4

Commit message: replicated h-bridges, added usb chip
Parts:
- added C10, C13, C16, C19: 100uF, adafruit:CPOL-US153CLV-0807
- added C11, C12, C14, C15, C17, C18, C20, C21, C22, C23: 1uF, adafruit:C-USC1206
- added D10, D11, D4, D5, D6, D7, D8, D9: BAV199, diode:BAV199
- added IC10: TUSB2046B, rov_club:TUSB2046B
- added IC6, IC7, IC8, IC9: VN5772AK, rov_club:VN5772AK
- added JP3, JP4, JP5, JP6: (no value), sparkfun:M02LOCK_LONGPADS
- added R10, R7, R8, R9: 10k, adafruit:R-US_R1206
- added U2: V_REG_LDOSMD, sparkfun:V_REG_LDOSMD
Connections:
- net SENSE renamed 0SENSE
- net STAT renamed 0STAT
- removed net 5H1: IC4.QA
- removed net 5H2: IC4.QB
- removed net 5H3: IC4.QC
- removed net 5H4: IC4.QD
- removed net H1: IC5.IN1
- removed net H2: IC5.IN2
- removed net H3: IC5.IN3
- removed net H4: IC5.IN4
- new net 0H1: IC2.QA, IC5.IN1
- new net 0H2: IC2.QB, IC5.IN2
- new net 0H3: IC2.QC, IC5.IN3
- new net 0H4: IC2.QD, IC5.IN4
- new net 1SENSE: IC6.SENSE, R7.1
- new net 1STAT: IC6.STAT3
- new net 2SENSE: IC7.SENSE, R8.1
- new net 2STAT: IC7.STAT3
- new net 3.3V: IC10.VCC@0, IC10.VCC@1, U2.OUT
- new net 3SENSE: IC8.SENSE, R9.1
- new net 3STAT: IC8.STAT3
- new net 4SENSE: IC9.SENSE, R10.1
- new net 4STAT: IC9.STAT3
- new net N$10: C12.2, D4.AC, IC6.DRAIN4@0, IC6.DRAIN4@1, IC6.DRAIN4@2, IC6.DRAIN4@3, IC6.SOURCE2@0, IC6.SOURCE2@1, JP3.2
- new net N$12: C15.1, D7.AC, IC7.DRAIN3@0, IC7.DRAIN3@1, IC7.DRAIN3@2, IC7.DRAIN3@3, IC7.SOURCE1@0, IC7.SOURCE1@1, JP4.1
- new net N$14: C15.2, D6.AC, IC7.DRAIN4@0, IC7.DRAIN4@1, IC7.DRAIN4@2, IC7.DRAIN4@3, IC7.SOURCE2@0, IC7.SOURCE2@1, JP4.2
- new net N$15: C18.1, D9.AC, IC8.DRAIN3@0, IC8.DRAIN3@1, IC8.DRAIN3@2, IC8.DRAIN3@3, IC8.SOURCE1@0, IC8.SOURCE1@1, JP5.1
- new net N$16: C18.2, D8.AC, IC8.DRAIN4@0, IC8.DRAIN4@1, IC8.DRAIN4@2, IC8.DRAIN4@3, IC8.SOURCE2@0, IC8.SOURCE2@1, JP5.2
- new net N$17: C21.1, D11.AC, IC9.DRAIN3@0, IC9.DRAIN3@1, IC9.DRAIN3@2, IC9.DRAIN3@3, IC9.SOURCE1@0, IC9.SOURCE1@1, JP6.1
- new net N$18: C21.2, D10.AC, IC9.DRAIN4@0, IC9.DRAIN4@1, IC9.DRAIN4@2, IC9.DRAIN4@3, IC9.SOURCE2@0, IC9.SOURCE2@1, JP6.2
- new net N$20: C23.1, U2.BP
- new net N$3: C12.1, D5.AC, IC6.DRAIN3@0, IC6.DRAIN3@1, IC6.DRAIN3@2, IC6.DRAIN3@3, IC6.SOURCE1@0, IC6.SOURCE1@1, JP3.1
- net +12V: now also C10.+, C11.1, C13.+, C14.1, C16.+, C17.1, C19.+, C20.1, D10.C, D11.C, D4.C, D5.C, D6.C, D7.C, D8.C, D9.C, IC6.VCC@0, IC6.VCC@1, IC6.VCC@2, IC6.VCC@3, IC7.VCC@0, IC7.VCC@1, IC7.VCC@2, IC7.VCC@3, IC8.VCC@0, IC8.VCC@1, IC8.VCC@2, IC8.VCC@3, IC9.VCC@0, IC9.VCC@1, IC9.VCC@2, IC9.VCC@3
- net +5V: now also C22.1, U2.EN, U2.IN
- net 1H1: now also IC2.QE, IC6.IN1; no longer IC2.QA
- net 1H2: now also IC2.QF, IC6.IN2; no longer IC2.QB
- net 1H3: now also IC2.QG, IC6.IN3; no longer IC2.QC
- net 1H4: now also IC2.QH, IC6.IN4; no longer IC2.QD
- net 2H1: now also IC3.QA, IC7.IN1; no longer IC2.QE
- net 2H2: now also IC3.QB, IC7.IN2; no longer IC2.QF
- net 2H3: now also IC3.QC, IC7.IN3; no longer IC2.QG
- net 2H4: now also IC3.QD, IC7.IN4; no longer IC2.QH
- net 3H1: now also IC3.QE, IC8.IN1; no longer IC3.QA
- net 3H2: now also IC3.QF, IC8.IN2; no longer IC3.QB
- net 3H3: now also IC3.QG, IC8.IN3; no longer IC3.QC
- net 3H4: now also IC3.QH, IC8.IN4; no longer IC3.QD
- net 4H1: now also IC4.QA, IC9.IN1; no longer IC3.QE
- net 4H2: now also IC4.QB, IC9.IN2; no longer IC3.QF
- net 4H3: now also IC4.QC, IC9.IN3; no longer IC3.QG
- net 4H4: now also IC4.QD, IC9.IN4; no longer IC3.QH
- net GND: now also C10.-, C11.2, C13.-, C14.2, C16.-, C17.2, C19.-, C20.2, C22.2, C23.2, D10.A, D11.A, D4.A, D5.A, D6.A, D7.A, D8.A, D9.A, IC6.GND, IC6.SOURCE3@0, IC6.SOURCE3@1, IC6.SOURCE4@0, IC6.SOURCE4@1, IC7.GND, IC7.SOURCE3@0, IC7.SOURCE3@1, IC7.SOURCE4@0, IC7.SOURCE4@1, IC8.GND, IC8.SOURCE3@0, IC8.SOURCE3@1, IC8.SOURCE4@0, IC8.SOURCE4@1, IC9.GND, IC9.SOURCE3@0, IC9.SOURCE3@1, IC9.SOURCE4@0, IC9.SOURCE4@1, R10.2, R7.2, R8.2, R9.2, U2.GND
Other:
- moved on the sheet: C9, IC4, X1A, X1B, X1C

Commit message: usb components
Parts:
- removed IC4: 74LS595D, sparkfun:74LS595D
- added C24, C25, C26, C27, C28, C29, C30, C31, C32: (no value), adafruit:C-USC1206
- added F1, F2, F3: (no value), dp_devices:FUSE_PTC-1812
- added JP7: (no value), sparkfun:M02LOCK_LONGPADS
- added R11, R12, R13, R14, R15, R16, R17, R18, R19, R20, R21, R22, R23, R24, R25, R26, R27, R28, R29: (no value), adafruit:R-US_R1206
- added U$1, U$2, U$3, U$4: TVS, sparkfun:TVS
- added Y2: 6MHz, sparkfun:RESONATORSMD
- C9: value 1uF -> (none)
- Y1: value RES -> 16Mhz
Connections:
- removed net 0H1: IC2.QA, IC5.IN1
- removed net 0H2: IC2.QB, IC5.IN2
- removed net 0H3: IC2.QC, IC5.IN3
- removed net 0H4: IC2.QD, IC5.IN4
- removed net 1H1: IC2.QE, IC6.IN1
- removed net 1H2: IC2.QF, IC6.IN2
- removed net 1H3: IC2.QG, IC6.IN3
- removed net 1H4: IC2.QH, IC6.IN4
- removed net 2H1: IC3.QA, IC7.IN1
- removed net 2H2: IC3.QB, IC7.IN2
- removed net 2H3: IC3.QC, IC7.IN3
- removed net 2H4: IC3.QD, IC7.IN4
- removed net 3H1: IC3.QE, IC8.IN1
- removed net 3H2: IC3.QF, IC8.IN2
- removed net 3H3: IC3.QG, IC8.IN3
- removed net 3H4: IC3.QH, IC8.IN4
- removed net 4H1: IC4.QA, IC9.IN1
- removed net 4H2: IC4.QB, IC9.IN2
- removed net 4H3: IC4.QC, IC9.IN3
- removed net 4H4: IC4.QD, IC9.IN4
- removed net RST: ISP1.RST, R1.1, U1.RESET/PC1
- removed net USB1+: X1A.2
- removed net USB1-: X1A.3
- removed net USB2+: X1B.2
- removed net USB2-: X1B.3
- removed net USB3+: X1C.2
- removed net USB3-: X1C.3
- new net !RST: IC10.!RST, ISP1.RST, R1.1, U1.RESET/PC1
- new net 0HA: IC2.QA, IC5.IN1, IC5.IN3
- new net 0HB: IC2.QB, IC5.IN2, IC5.IN4
- new net 1HA: IC2.QC, IC6.IN1, IC6.IN3
- new net 1HB: IC2.QD, IC6.IN2, IC6.IN4
- new net 2HA: IC2.QE, IC7.IN1, IC7.IN3
- new net 2HB: IC2.QF, IC7.IN2, IC7.IN4
- new net 3HA: IC2.QG, IC8.IN1, IC8.IN3
- new net 3HB: IC2.QH, IC8.IN2, IC8.IN4
- new net 4HA: IC3.QA, IC9.IN1, IC9.IN3
- new net 4HB: IC3.QB, IC9.IN2, IC9.IN4
- new net 5HA: IC3.QC
- new net 5HB: IC3.QD
- new net N$19: C24.1, IC10.D0+, R11.1, R12.1, U$1.2
- new net N$21: R15.1, R21.1, U$2.1, X1C.2
- new net N$22: IC10.XTAL1, Y2.3
- new net N$23: IC10.XTAL2, Y2.1
- new net N$24: R14.1, R20.1, U$2.2, X1C.3
- new net N$25: R19.1, R22.1, U$3.2, X1B.3
- new net N$26: C30.1, IC10.D2+, R16.2
- new net N$27: C29.1, IC10.D2-, R17.2
- new net N$28: C28.1, IC10.D3+, R18.2
- new net N$29: C27.1, IC10.D3-, R19.2
- new net N$30: C25.1, IC10.D4-, R20.2
- new net N$31: C26.1, IC10.D4+, R21.2
- new net N$32: R18.1, R23.1, U$3.1, X1B.2
- new net N$33: R17.1, R24.1, U$4.2, X1A.3
- new net N$34: R16.1, R25.1, U$4.1, X1A.2
- new net N$35: F1.2, X1C.1
- new net N$36: F2.2, X1B.1
- new net N$37: F3.2, X1A.1
- new net N$38: R27.2, R29.1
- new net N$39: IC10.D1-
- new net N$40: IC10.D1+
- new net N$41: C32.1, R26.1, U1.D+
- new net N$42: C31.1, R27.1, U1.D-
- new net N$43: R26.2, R28.1
- new net N$44: JP7.1, R12.2
- new net N$45: JP7.2, R13.2
- net !CLR: no longer IC4.SCL
- net +5V: now also F1.1, F2.1, F3.1; no longer C9.1, IC4.VCC, X1A.1, X1B.1, X1C.1
- net 3.3V: now also IC10.!EXTMEM, IC10.!OVRCUR1, IC10.!OVRCUR2, IC10.!OVRCUR3, IC10.!OVRCUR4, R11.2
- net GND: now also C24.2, C25.2, C26.2, C27.2, C28.2, C29.2, C30.2, C31.2, C32.2, IC10.BUSPWR, IC10.EEDATA/GANGED, IC10.GND@0, IC10.GND@1, IC10.PLL/48M, IC10.TSTMODE, R14.2, R15.2, R22.2, R23.2, R24.2, R25.2, R28.2, R29.2, Y2.2; no longer IC4.G, IC4.GND
- net N$7: now also C9.1, IC10.D0-, R13.1, U$1.1; no longer IC3.QH*, IC4.SER
- net RCK: no longer IC4.RCK
- net SCK: no longer IC4.SCK
Other:
- moved on the sheet: C1, C16, C17, C18, C19, C2, C20, C21, C22, C23, C7, C8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

Commit message: replacing usb enabled uC with two chip solution
Parts:
- removed C32: (no value), adafruit:C-USC1206
- removed R27, R28, R29: (no value), adafruit:R-US_R1206
- removed U1: ATMEGA8U2AU, sparkfun:ATMEGA8U2AU
- added U3: ATMEGA168, sparkfun:ATMEGA168
- added ZD2: (no value), dp_devices:ZENERSOD-123
Connections:
- net N$39 renamed D1-
- net N$40 renamed D1+
- removed net N$38: R27.2, R29.1
- removed net N$41: C32.1, R26.1, U1.D+
- removed net N$42: C31.1, R27.1, U1.D-
- removed net N$43: R26.2, R28.1
- new net !USB_RST: R26.2
- new net AGND: U3.AGND
- new net RXD: U3.PD0(RXD)
- new net TXD: U3.PD1(TXD)
- net !RST: now also U3.PC6(/RESET); no longer IC10.!RST, U1.RESET/PC1
- net +5V: now also C3.1, C31.1, U3.AREF, U3.AVCC, U3.VCC@1, U3.VCC@2; no longer U1.AVCC, U1.UVCC, U1.VCC
- net 0SENSE: now also U3.PC0(ADC0)
- net 1SENSE: now also U3.PC1(ADC1)
- net 2SENSE: now also U3.PC2(ADC2)
- net 3SENSE: now also U3.PC3(ADC3)
- net 4SENSE: now also U3.PC4(ADC4/SDA)
- net GND: now also U3.GND@1, U3.GND@2, ZD2.A; no longer C32.2, R28.2, R29.2, U1.GND, U1.UGND
- net ISP-MISO: now also U3.PB4(MISO); no longer U1.PB3(MISO)
- net ISP-MOSI: now also U3.PB3(MOSI/OC2); no longer U1.PB2(MOSI)
- net ISP-SCK: now also U3.PB5(SCK); no longer U1.PB1(SCK)
- net N$2: now also U3.PB7(XTAL2/TOSC2); no longer U1.XTAL2/PC0
- net N$4: now also U3.PB6(XTAL1/TOSC1); no longer U1.XTAL1
- net N$5: now also IC10.!RST, R26.1, ZD2.C; no longer C3.1, U1.UCAP
Other:
- moved on the sheet: C1, C10, C11, C12, C13, C14, C15, C16, C17, C18, C19, C2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

Commit message: added usb/ttl
Parts:
- removed Q2: BSS84, transistor-small-signal:BSS84
- removed X1: USB_3PSHIELD-85-32003-00X-1, con-cypressindustries:USB_3PSHIELD-85-32003-00X-1
- added C32, C33, C34, C35, C36: (no value), adafruit:C-USC1206
- added IC4: IC_FT230X-SSOP-16, dp_devices:IC_FT230X-SSOP-16
- added JP10, JP8, JP9: (no value), sparkfun:M04SCREW
- added L2, L3, L4: (no value), sparkfun:INDUCTOR1206H*
- added LED1, LED2: (no value), adafruit:LEDCHIPLED_1206
- added Q1: FDD4141TO252, transistor-fet:FDD4141TO252
- added R27, R28, R29, R30, R31, R32: (no value), adafruit:R-US_R1206
- JP2, JP3, JP4, JP5, JP6, JP7: device sparkfun:M02LOCK_LONGPADS -> sparkfun:M023.5MM
Connections:
- removed net !CLR: IC2.SCL, IC3.SCL
- removed net RCK: IC2.RCK, IC3.RCK
- new net ARM_EN: U3.PB1(OC1A)
- new net CONDUCT: U3.ADC7
- new net LATCH: IC2.RCK, IC3.RCK, U3.PB2(SS/OC1B)
- new net N$38: IC4.!RESET, IC4.3V3OUT, IC4.VCCIO, R31.1, R32.1
- new net N$39: IC4.USB-, R27.2, R28.2
- new net N$40: IC4.USB+, R29.2, R30.2
- new net N$41: F3.1, L2.2
- new net N$42: F2.1, L3.2
- new net N$43: IC3.QH
- new net N$46: IC3.QG
- new net N$47: IC3.QF
- new net N$48: IC3.QE
- new net N$49: F1.1, L4.2
- new net N$50: IC4.CBUS1, LED1.C
- new net N$51: IC4.CBUS2, LED2.C
- new net N$52: LED1.A, R31.2
- new net N$53: LED2.A, R32.2
- new net RANG_EN: U3.PB0(ICP)
- new net TEMP0: U3.PC5(ADC5/SCL)
- new net TEMP1: U3.ADC6
- net !RST: now also IC4.!RTS
- net !USB_RST: now also U3.PD7(AIN1)
- net +12V: now also Q1.S; no longer Q2.S
- net +5V: now also C34.1, IC2.SCL, IC3.SCL, IC4.VCC, L2.1, L3.1, L4.1; no longer F1.1, F2.1, F3.1
- net 0STAT: now also U3.PD2(INT0)
- net 1STAT: now also U3.PD3(INT1)
- net 2STAT: now also U3.PD4(XCK/T0)
- net 3.3V: now also C35.1, C36.1
- net 3STAT: now also U3.PD5(T1)
- net 4STAT: now also U3.PD6(AIN0)
- net D1+: now also C32.1, R29.1
- net D1-: now also C33.1, R28.1
- net GND: now also C32.2, C33.2, C34.2, C35.2, C36.2, IC4.GND@1, IC4.GND@2, JP10.4, JP8.4, JP9.4, R27.1, R30.1; no longer X1A.4, X1B.4, X1C.4
- net N$21: now also JP10.3; no longer X1C.2
- net N$24: now also JP10.2; no longer X1C.3
- net N$25: now also JP9.2; no longer X1B.3
- net N$32: now also JP9.3; no longer X1B.2
- net N$33: now also JP8.2; no longer X1A.3
- net N$34: now also JP8.3; no longer X1A.2
- net N$35: now also JP10.1; no longer X1C.1
- net N$36: now also JP9.1; no longer X1B.1
- net N$37: now also JP8.1; no longer X1A.1
- net N$8: now also Q1.D; no longer Q2.D
- net N$9: now also Q1.G; no longer Q2.G
- net RXD: now also IC4.TXD
- net TXD: now also IC4.RXD
Other:
- moved on the sheet: C1, C2, C22, C23, C24, C25, C26, C27, C28, C29, C3, C30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

Commit message: rearranged some signals, corrected cap values
Parts:
- removed Q1: FDD4141TO252, transistor-fet:FDD4141TO252
- removed R5: 100k, adafruit:R-US_R1206
- removed ZD1: (no value), dp_devices:ZENERSOD-123
- added C37, C38, C39, C40, C41, C42: 4.7uF, adafruit:C-USC1206
- C1, C10, C13, C16, C19, C4: value 100uF -> 1000uF
- C11, C14, C17, C20, C5, C7, C8: value 1uF -> 0.1uF
- C22: value 1uF -> 4.7uF
- F1, F2, F3: value (none) -> 500mA
Connections:
- removed net N$8: JP1.2, Q1.D
- removed net N$9: Q1.G, R5.1, ZD1.A
- net +12V: now also C38.1, C39.1, C40.1, C41.1, C42.1, JP1.2; no longer Q1.S, ZD1.C
- net +5V: now also C37.1
- net GND: now also C37.2, C38.2, C39.2, C40.2, C41.2, C42.2; no longer R5.2
Other:
- moved on the sheet: C1, C10, C11, C12, C13, C14, C15, C16, C17, C18, C19, C2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

Commit message: working on conductivity sensor circuit
Parts:
- added C43, C44, C45: (no value), adafruit:C-USC1206
- added F4: 500mA, dp_devices:FUSE_PTC-1812
- added IC11: OPA129U, burr-brown:OPA129U
- added JP11: (no value), sparkfun:M023.5MM
- added R33, R5: (no value), adafruit:R-US_R1206
- added U$5: TVS, sparkfun:TVS
Connections:
- new net N$8: F4.1, R5.1
- new net N$9: C45.1, IC11.+IN, JP11.1, R33.1, R5.2, U$5.2
- net +5V: now also C43.1, C44.1, F4.2, IC11.V+
- net AGND: now also C43.2, C44.2, C45.2, IC11.V-, JP11.2, R33.2, U$5.1
- net CONDUCT: now also IC11.-IN, IC11.OUT
