File: motherboard.brd (EAGLE design)
At the start: 177.1 x 75.9 mm, 215 parts, among them IC1 LM2576, IC10 TUSB2046B, IC12 LM50, IC13 LM50, IC2 74LS595D, IC3 74LS595D, IC4 IC_FT230X-SSOP-16, IC5 VN5772AK, IC6 VN5772AK, IC7 VN5772AK, IC8 VN5772AK, IC9 VN5772AK, U2 NCP4625, U3 ATMEGA168, Y1 16Mhz, Y2 6MHz

Commit message: layed out hbridges, MCU, new fuses
Parts:
- removed C44, C45, C56: 1000uF, adafruit:153CLV-0807
- removed F5, F6, F7: (no value), special:FUSE1
- removed JP10, JP9: (no value), sparkfun:SCREWTERMINAL-3.5MM-4
- removed JP7: (no value), sparkfun:SCREWTERMINAL-3.5MM-2
- removed L1: 100uH, sparkfun:INDUCTOR-1206
- removed Q4, Q5, Q6: (no value), adafruit:SOT23
- removed U$19, U$20, U$9: TVS, sparkfun:SMA-DIODE
- added JP13: (no value), sparkfun:SCREWTERMINAL-3.5MM-4
- added L18: 100uH, sparkfun:CDRH125
- F4, F8, F9: value (none) -> 3557-2; device special:FUSE1 -> rov_club:3557-2
- JP11, JP17: device sparkfun:SCREWTERMINAL-3.5MM-2 -> sparkfun:SCREWTERMINAL-3.5MM-4
- JP12: device sparkfun:SCREWTERMINAL-3.5MM-2 -> sparkfun:1X03
- JP8: device sparkfun:SCREWTERMINAL-3.5MM-4 -> sparkfun:SCREWTERMINAL-3.5MM-2
- moved C12 487.5 mm to (134.0, -36.8)
- moved C6 487.5 mm to (122.9, -36.8)
- moved D2 487.5 mm to (121.0, -30.5)
- moved D3 487.5 mm to (121.0, -21.6)
- moved D4 487.5 mm to (124.8, -30.5)
- moved D5 487.5 mm to (124.8, -21.6)
- moved D6 487.5 mm to (132.1, -30.5)
- moved D7 487.5 mm to (132.1, -21.6)
- moved D8 487.5 mm to (135.9, -30.5)
- moved D9 487.5 mm to (135.9, -21.6)
- moved R5 487.4 mm to (152.4, 28.9), turned to 0 degrees
- moved R6 486.5 mm to (152.4, 26.4), turned to 0 degrees
- moved ZD1 484.0 mm to (148.0, 27.3), turned to 90 degrees
- moved C38 480.1 mm to (158.8, 27.6)
- moved C4 480.1 mm to (170.2, 19.1)
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Connections:
- removed net N$20: C56.+, F8.1A, JP17.1, U$9.C
- removed net N$57: JP17.2, Q4.3
- removed net N$72: JP11.2, Q5.3
- removed net N$73: JP12.2, Q6.3
- removed net N$74: C45.+, F9.1A, JP12.1, U$20.C
- removed net N$75: C44.+, F4.1A, JP11.1, U$19.C
- net +12V: now also F4.P$3, F4.P$4, F8.P$3, F8.P$4, F9.P$3, F9.P$4; no longer F4.2A, F5.2A, F6.2A, F7.2A, F8.2A, F9.2A
- net +5V: now also L18.2; no longer L1.P$2
- net GND: now also JP11.1, JP13.1, JP17.1; no longer C44.-, C45.-, C56.-, JP10.4, JP8.4, JP9.4, Q4.2, Q5.2, Q6.2, U$19.A, U$20.A, U$9.A
- net N$1: now also L18.1; no longer L1.P$1
- net N$21: now also JP17.2; no longer JP10.3
- net N$24: now also JP17.3; no longer JP10.2
- net N$25: now also JP13.3; no longer JP9.2
- net N$32: now also JP13.2; no longer JP9.3
- net N$33: now also JP11.3; no longer JP8.2
- net N$34: now also JP11.2; no longer JP8.3
- net N$35: now also JP17.4; no longer JP10.1
- net N$36: now also JP13.4; no longer JP9.1
- net N$37: now also JP11.4; no longer JP8.1
- net N$43: now also JP14.1; no longer JP14.2
- net N$44: now also JP8.1; no longer JP7.1
- net N$45: now also JP8.2; no longer JP7.2
- net N$47: now also JP15.1; no longer JP15.2
- net N$48: now also JP16.1; no longer JP16.2
- net N$50: now also F9.P$1, F9.P$2, JP16.2; no longer F7.1A, JP16.1
- net N$54: now also F8.P$1, F8.P$2, JP15.2; no longer F6.1A, JP15.1
- net N$55: now also F4.P$1, F4.P$2, JP14.2; no longer F5.1A, JP14.1
- net SW3: now also JP12.1; no longer Q4.1
- net SW4: now also JP12.2; no longer Q5.1
- net SW5: now also JP12.3; no longer Q6.1
Routing:
- net +12V: track 370.2 -> 309.8 mm
- net AGND: track 18.3 -> 54.5 mm
- net N$75: track 22.3 -> 0.00 mm
- net N$74: track 22.3 -> 0.00 mm
- net N$20: track 22.3 -> 0.00 mm
- net GND: track 95.5 -> 74.4 mm
- net +5V: track 160.4 -> 179.8 mm
- net N$13: track 72.8 -> 58.0 mm
- net N$59: track 74.0 -> 60.5 mm
- net !RST: track 0.00 -> 12.8 mm
- net N$3: track 68.7 -> 58.0 mm
- net N$5: track 70.2 -> 60.5 mm
- net N$1: track 9.43 -> 19.1 mm
- net ISP-MOSI: track 0.00 -> 9.68 mm
- net D1-: track 26.0 -> 35.6 mm
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
Commit message: positioned all but mcu
Parts:
- removed R40, R42, R43, R44, R45, R46, R47, R48, R49, R50, R51, R52, R53, R54, R55, R56: 10k, adafruit:R1206
- added R41, R57: 10k, resistor-bourns:SO16
- D10, D11, D12, D13, D14, D15, D16, D17, D18, D19, D2, D20, D21, D3, D4, D5, D6, D7, D8, D9: device adafruit:SMADIODE -> adafruit:SOD-123
- moved C48 336.3 mm to (173.0, 17.1), turned to 180 degrees
- moved C49 332.9 mm to (173.0, 19.7), turned to 180 degrees
- moved IC13 328.6 mm to (173.0, 22.9), turned to 90 degrees
- moved F4 325.4 mm to (77.5, 35.6), turned to 90 degrees
- moved C51 324.3 mm to (173.0, 26.0), turned to 180 degrees
- moved U$6 319.4 mm to (79.4, 12.7), turned to 0 degrees
- moved C53 319.3 mm to (77.5, 20.3), turned to 90 degrees
- moved Q1 312.4 mm to (74.3, 12.7), turned to 180 degrees
- moved F8 311.8 mm to (67.3, 35.6), turned to 90 degrees
- moved JP14 308.6 mm to (72.1, 6.67), turned to 0 degrees
- moved C54 305.4 mm to (67.3, 20.3), turned to 90 degrees
- moved U$7 305.4 mm to (69.2, 12.7), turned to 0 degrees
- moved Q2 298.4 mm to (64.1, 12.7), turned to 180 degrees
- moved F9 298.3 mm to (57.1, 35.6), turned to 90 degrees
- moved JP15 297.5 mm to (65.1, 6.67), turned to 0 degrees
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Connections:
- net 0HA: now also R41.3; no longer R40.1
- net 0HB: now also R41.1; no longer R42.1
- net 1HA: now also R41.2; no longer R43.1
- net 1HB: now also R41.4; no longer R44.1
- net 2HA: now also R41.5; no longer R45.1
- net 2HB: now also R41.6; no longer R46.1
- net 3HA: now also R41.7; no longer R47.1
- net 3HB: now also R41.8; no longer R48.1
- net 4HA: now also R57.3; no longer R49.1
- net 4HB: now also R57.1; no longer R50.1
- net N$10: now also JP5.1; no longer JP5.2
- net N$11: now also JP5.2; no longer JP5.1
- net N$12: now also JP6.1; no longer JP6.2
- net N$13: now also JP2.1; no longer JP2.2
- net N$14: now also JP6.2; no longer JP6.1
- net N$15: now also R57.9; no longer R56.2
- net N$17: now also R57.10; no longer R55.2
- net N$18: now also R57.11; no longer R54.2
- net N$3: now also JP3.1; no longer JP3.2
- net N$5: now also JP3.2; no longer JP3.1
- net N$56: now also R57.12; no longer R53.2
- net N$59: now also JP2.2; no longer JP2.1
- net N$60: now also R57.13; no longer R52.2
- net N$61: now also R57.15; no longer R51.2
- net N$62: now also R57.16; no longer R50.2
- net N$63: now also R57.14; no longer R49.2
- net N$64: now also R41.9; no longer R48.2
- net N$65: now also R41.10; no longer R47.2
- net N$66: now also R41.11; no longer R46.2
- net N$67: now also R41.12; no longer R45.2
- net N$68: now also R41.13; no longer R44.2
- net N$69: now also R41.15; no longer R43.2
- net N$70: now also R41.16; no longer R42.2
- net N$71: now also R41.14; no longer R40.2
- net N$8: now also JP4.1; no longer JP4.2
- net N$9: now also JP4.2; no longer JP4.1
- net SW0: now also R57.2; no longer R51.1
- net SW1: now also R57.4; no longer R52.1
- net SW2: now also R57.5; no longer R53.1
- net SW3: now also R57.6; no longer R54.1
- net SW4: now also R57.7; no longer R55.1
- net SW5: now also R57.8; no longer R56.1
Routing:
- net GND: track 74.4 -> 12.1 mm, vias 279 -> 275
- net N$14: track 69.2 -> 32.3 mm
- net +12V: track 309.8 -> 343.9 mm, vias 5 -> 10
- net N$12: track 66.3 -> 32.3 mm
- net N$11: track 67.4 -> 33.6 mm
- net N$10: track 64.6 -> 32.3 mm
- net N$9: track 61.8 -> 32.6 mm
- net N$59: track 60.5 -> 32.3 mm
- net N$5: track 60.5 -> 32.3 mm
- net N$8: track 59.2 -> 32.6 mm
- net N$3: track 58.0 -> 32.3 mm
- net N$13: track 58.0 -> 32.3 mm
- net N$63: track 2.80 -> 13.4 mm, vias 0 -> 2
- net N$55: track 21.6 -> 30.1 mm
- net N$71: track 2.66 -> 10.7 mm, vias 0 -> 2
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
Commit message: putting things into place
Routing:
- net +12V: track 343.9 -> 535.6 mm
- net N$14: track 32.3 -> 59.5 mm
- net N$5: track 32.3 -> 59.0 mm
- net N$13: track 32.3 -> 58.9 mm
- net N$12: track 32.3 -> 58.1 mm
- net N$3: track 32.3 -> 57.6 mm
- net N$59: track 32.3 -> 57.3 mm
- net N$11: track 33.6 -> 41.6 mm
- net N$10: track 32.3 -> 40.0 mm
- net N$9: track 32.6 -> 39.1 mm
- net N$8: track 32.6 -> 39.0 mm

Commit message: layed out control lines to hbridges, fets
Parts:
- moved JP12 150.8 mm to (81.9, 72.4), turned to 0 degrees
- moved IC3 38.1 mm to (74.0, 69.2)
- moved C37 38.1 mm to (51.4, 69.2)
- moved C7 38.1 mm to (54.0, 69.2)
- moved C8 38.1 mm to (67.3, 69.2)
- moved R41 38.1 mm to (60.0, 61.6)
- moved R57 38.1 mm to (73.3, 61.6)
- moved IC2 38.1 mm to (60.6, 69.2)
- moved ISP2 32.4 mm to (23.5, 69.8)
- moved ISP5 32.4 mm to (42.5, 69.8)
- moved R2 32.4 mm to (14.6, 63.5)
- moved R32 32.4 mm to (23.5, 59.7)
- moved R39 32.4 mm to (42.5, 59.7)
- moved R4 32.4 mm to (14.6, 69.8)
- moved U$11 32.4 mm to (47.6, 63.5)
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Connections:
- net 0HA: now also IC6.2, IC6.8, R41.2; no longer IC5.2, IC5.8, R41.3
- net 0HB: now also IC6.13, IC6.7; no longer IC5.13, IC5.7
- net 0SENSE: now also R8.1, R9.1, ZD2.C; no longer R5.1, R6.1, ZD1.C
- net 0STAT: now also IC6.4; no longer IC5.4
- net 1HA: now also R41.3; no longer R41.2
- net 2HA: now also IC5.2, IC5.8; no longer IC6.2, IC6.8
- net 2HB: now also IC5.13, IC5.7; no longer IC6.13, IC6.7
- net 2SENSE: now also R5.1, R6.1, ZD1.C; no longer R8.1, R9.1, ZD2.C
- net 2STAT: now also IC5.4; no longer IC6.4
- net N$69: now also R41.14; no longer R41.15
- net N$71: now also R41.15; no longer R41.14
- net SW0: now also Q3.1; no longer Q1.1
- net SW2: now also Q1.1; no longer Q3.1
Routing:
- net 3HB: track 13.0 -> 119.3 mm, vias 2 -> 3
- net 2HA: track 16.8 -> 122.0 mm, vias 2 -> 3
- net 3HA: track 16.8 -> 115.0 mm, vias 2 -> 3
- net 2HB: track 13.0 -> 110.0 mm, vias 2 -> 3
- net 1HA: track 16.8 -> 97.7 mm, vias 2 -> 3
- net 4HB: track 13.0 -> 92.7 mm, vias 2 -> 3
- net SW2: track 0.00 -> 77.0 mm
- net 1HB: track 13.0 -> 86.1 mm, vias 2 -> 3
- net SW1: track 0.00 -> 68.4 mm
- net 0HA: track 17.0 -> 80.3 mm, vias 2 -> 3
- net SW0: track 0.00 -> 62.8 mm
- net 4HA: track 17.0 -> 76.1 mm, vias 2 -> 3
- net +12V: track 535.6 -> 592.5 mm
- net 0HB: track 13.0 -> 60.1 mm, vias 2 -> 3
- net +5V: track 181.9 -> 207.5 mm
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Other:
- outline, holes or cut-outs redrawn
