File: production.brd (EAGLE design)
At the start: 177.2 x 153.4 mm, 362 parts, among them IC1 LM2576, IC10 TUSB2046B, IC11 LM2576, IC12 LM50, IC13 LM50, IC14 74LS595D, IC15 74LS595D, IC16 VN5772AK, IC17 TUSB2046B, IC18 IC_FT230X-SSOP-16, IC19 LM50, IC2 74LS595D, IC20 LM50, IC21 VN5772AK, IC22 VN5772AK, IC23 VN5772AK, IC24 VN5772AK, IC3 74LS595D, IC4 IC_FT230X-SSOP-16, IC5 VN5772AK, IC6 VN5772AK, IC7 VN5772AK, IC8 VN5772AK, IC9 VN5772AK, U1 NCP4625, U2 NCP4625, U3 ATMEGA168, U4 ATMEGA168, Y1 16Mhz, Y2 6MHz, Y3 16Mhz, Y4 6MHz

Commit message: tweaks to boards
Routing:
- net GND1: vias 368 -> 364
- net GND: vias 368 -> 364
Changed lines of the file:
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@@
 <via x="85.4075" y="52.07" extent="1-16" drill="0.5"/>
 <via x="85.4075" y="50.8" extent="1-16" drill="0.5"/>
-<via x="85.4075" y="49.53" extent="1-16" drill="0.5"/>
-<via x="85.4075" y="48.26" extent="1-16" drill="0.5"/>
-<via x="85.4075" y="46.99" extent="1-16" drill="0.5"/>
-<via x="85.4075" y="54.61" extent="1-16" drill="0.5"/>
 <via x="86.6775" y="53.34" extent="1-16" drill="0.5"/>
 <via x="86.6775" y="52.07" extent="1-16" drill="0.5"/>
@@
 <via x="85.4075" y="129.54" extent="1-16" drill="0.5"/>
 <via x="85.4075" y="128.27" extent="1-16" drill="0.5"/>
-<via x="85.4075" y="127" extent="1-16" drill="0.5"/>
-<via x="85.4075" y="125.73" extent="1-16" drill="0.5"/>
-<via x="85.4075" y="124.46" extent="1-16" drill="0.5"/>
-<via x="85.4075" y="132.08" extent="1-16" drill="0.5"/>
 <via x="86.6775" y="130.81" extent="1-16" drill="0.5"/>
 <via x="86.6775" y="129.54" extent="1-16" drill="0.5"/>
